File: pcb/usb2can.sch (EAGLE design)
At the start: 48 parts, among them CON1 USB_A_MALESMD, IC1 ADM3053M, IC2 LD1117S33

Commit message: pcb: adapt resistor values for LEDs
Parts:
- R10: value 330R -> 270R
- R7, R9: value 33R -> 120R
Changed lines of the file:
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@@
 <part name="LED2" library="led" deviceset="LED" device="CHIPLED_0603" value="BLUE"/>
 <part name="+3V9" library="supply1" deviceset="+3V3" device=""/>
-<part name="R7" library="resistor" deviceset="R-EU_" device="R0603" value="33R"/>
+<part name="R7" library="resistor" deviceset="R-EU_" device="R0603" value="120R"/>
 <part name="S3" library="micro_switch" deviceset="MICRO_SWITCH_3X6X2.5" device="S"/>
 <part name="GND20" library="supply1" deviceset="GND" device=""/>
@@
 <part name="LED4" library="led" deviceset="LED" device="CHIPLED_0603" value="WHITE"/>
 <part name="+3V11" library="supply1" deviceset="+3V3" device=""/>
-<part name="R9" library="resistor" deviceset="R-EU_" device="R0603" value="33R"/>
+<part name="R9" library="resistor" deviceset="R-EU_" device="R0603" value="120R"/>
 <part name="LED5" library="led" deviceset="LED" device="CHIPLED_0603" value="GREEN"/>
 <part name="+3V12" library="supply1" deviceset="+3V3" device=""/>
-<part name="R10" library="resistor" deviceset="R-EU_" device="R0603" value="330R"/>
+<part name="R10" library="resistor" deviceset="R-EU_" device="R0603" value="270R"/>
 <part name="TP3" library="testpad" deviceset="TPS" device="TP07R" value="TPSTP07R"/>
 <part name="C20" library="rcl" deviceset="C-EU" device="C0603" value="100n"/>
