File: pcb/usb2can.sch (EAGLE design)
At the start: 48 parts, among them CON1 USB_A_MALESMD, IC1 ADM3053M, IC2 LD1117S33

Commit message: schematic: rename unnamed wires to CANH and CANL.
Connections:
- net N$2 renamed CANL
- net N$3 renamed CANH
Changed lines of the file:
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@@
 </segment>
 </net>
-<net name="N$2" class="0">
+<net name="CANL" class="0">
 <segment>
 <pinref part="IC1" gate="G$1" pin="CAN_L"/>
@@
 </segment>
 </net>
-<net name="N$3" class="0">
+<net name="CANH" class="0">
 <segment>
 <pinref part="IC1" gate="G$1" pin="CAN_H"/>
